Commit message: modified two joint snake and added launch file and using bash to launch rviz

File: snake_description/urdf/twoJoints.urdf (robot description, URDF)
Before this commit: robot twoJointsSnake, 2 links, 1 joints
Links:
- removed link link1
- added link base_link; visual mesh filename=package://snake_robot/snake_description/meshes/servo.stl scale=0.001 0.001 0.001
- link link2: geometry visual mesh filename=package://snake_robot/snake_description/meshes/servo.stl scale=0.001 0.001 0.001
Joints:
- joint joint1: parent link1 -> base_link

Commit message: fix joint2 rotate axis by turn the joint 90 degree

File: snake_description/urdf/twoJoints.urdf (robot description, URDF)
Before this commit: robot twoJointsSnake, 2 links, 1 joints
Links:
- added link link3; visual mesh filename=package://snake_robot/snake_description/meshes/servo.stl scale=0.001 0.001 0.001
Joints:
- added joint joint2: type continuous, parent link2, child link3, origin xyz=0. 0. 0. rpy=0. 0. 1.57079632679

Commit message: show path for end link

File: snake_description/urdf/twoJoints.urdf (robot description, URDF)
Before this commit: robot twoJointsSnake, 3 links, 2 joints
Joints:
- joint joint2: origin xyz=0. 0. 0. rpy=0. 0. 1.57079632679 -> xyz=0. 0. 0.06 rpy=0. 0. 1.57079632679

Commit message: correct the real model by change size and joint limit

File: snake_description/urdf/twoJoints.urdf (robot description, URDF)
Before this commit: robot twoJointsSnake, 3 links, 2 joints
Joints:
- joint joint1: limit (none) -> lower=-1 upper=1 effort=0.01 velocity=0.5; origin (none) -> xyz=0. 0. 0. rpy=0. 0. 0.
- joint joint2: limit (none) -> lower=-1 upper=1 effort=0.01 velocity=0.5; origin xyz=0. 0. 0.06 rpy=0. 0. 1.57079632679 -> xyz=0. 0. 0.072 rpy=0. 0. 1.57079632679

Commit message: added new demo, using ros control to simulation in gazebo

File: snake_description/urdf/twoJoints.urdf (robot description, URDF)
Before this commit: robot twoJointsSnake, 3 links, 2 joints
Links:
- added link world
- link base_link: mass None -> 1
- link link2: mass None -> 1
- link link3: mass None -> 1
Joints:
- added joint fixed: type fixed, parent world, child base_link
