Commit message: added three joint

File: snake_description/urdf/threeJoints.urdf (robot description, URDF)
Before this commit: robot twoJointsSnake, 3 links, 2 joints
Links:
- added link link4; visual mesh filename=package://snake_robot/snake_description/meshes/servo.stl scale=0.001 0.001 0.001
Joints:
- added joint joint3: type continuous, parent link3, child link4, origin xyz=0. 0. 0.072 rpy=0. 0. 0., limit lower=-1 upper=1 effort=0.01 velocity=0.5

Commit message: added launch to draw circle using seven joint snake

File: snake_description/urdf/threeJoints.urdf (robot description, URDF)
Before this commit: robot threeJointsSnake, 5 links, 4 joints
Links:
- link link4: mass None -> 1
